File: monitoring_board/monitoring_board.kicad_pcb (KiCad board)
At the start: 2 copper layers, 101.6 x 53.3 mm, 13 parts, among them P1 Digital, P10 CONN_01X01, P11 CONN_01X01, P12 CONN_01X01, P13 CONN_01X01, P2 Power, P3 Analog, P4 Analog, P5 PWM, P6 PWM, P7 Communication, P8 CONN_01X01, P9 CONN_01X01

Commit message: Monitoring board: start pcb design
Parts:
- added D3: LED, LEDs:LED_D5.0mm, F.Cu at (131.6, 30.5)
- added D4: LED, LEDs:LED_D5.0mm, F.Cu at (143.8, 30.5)
- added D5: LED, LEDs:LED_D5.0mm, F.Cu at (177.0, 21.3)
- added D6: LED, LEDs:LED_D5.0mm, F.Cu at (-25.7, 167.4)
- added D7: LED, LEDs:LED_D5.0mm, F.Cu at (164.8, 18.3)
- added D8: LED, LEDs:LED_D5.0mm, F.Cu at (171.4, 29.2)
- added D9: LED, LEDs:LED_D5.0mm, F.Cu at (154.2, 30.0)
- added DS1: WC1602A, Displays:WC1602A, F.Cu at (57.8, -48.2)
- added F1: 30A Polyfuse, Fuse_Holders_and_Fuses:Fuse_TE5_Littlefuse-395Series, F.Cu at (59.8, 126.5)
- added F2: 4A Polyfuse, Fuse_Holders_and_Fuses:Fuse_TE5_Littlefuse-395Series, F.Cu at (79.9, 53.6)
- added J1: Conn_01x02, Connectors_Terminal_Blocks:TerminalBlock_bornier-2_P5.08mm, F.Cu at (79.8, 129.5)
- added J10: Conn_01x02, Connectors_Terminal_Blocks:TerminalBlock_bornier-2_P5.08mm, F.Cu at (234.4, 101.0)
- added J11: Conn_01x02, Connectors_Terminal_Blocks:TerminalBlock_bornier-2_P5.08mm, F.Cu at (234.4, 114.2)
- added J12: Conn_01x02, Connectors_Terminal_Blocks:TerminalBlock_bornier-2_P5.08mm, F.Cu at (234.4, 127.5)
- added J13: Conn_01x02, Connectors_Terminal_Blocks:TerminalBlock_bornier-2_P5.08mm, F.Cu at (234.4, 140.7)
- added J2: Conn_01x02, Connectors_Terminal_Blocks:TerminalBlock_bornier-2_P5.08mm, F.Cu at (59.9, 50.5)
- added J3: Conn_01x02, Connectors_Terminal_Blocks:TerminalBlock_bornier-2_P5.08mm, F.Cu at (234.4, 48.0)
- added J4: Conn_01x02, Connectors_Terminal_Blocks:TerminalBlock_bornier-2_P5.08mm, F.Cu at (215.9, 139.2)
- added J5: Conn_01x05, Pin_Headers:Pin_Header_Straight_1x05_Pitch2.54mm, F.Cu at (181.1, 49.5)
- added J6: Conn_02x08_Odd_Even, Pin_Headers:Pin_Header_Straight_2x08_Pitch2.54mm, F.Cu at (161.8, 47.0)
- added J7: Conn_01x02, Connectors_Terminal_Blocks:TerminalBlock_bornier-2_P5.08mm, F.Cu at (234.4, 61.3)
- added J8: Conn_01x02, Connectors_Terminal_Blocks:TerminalBlock_bornier-2_P5.08mm, F.Cu at (234.4, 74.5)
- added J9: Conn_01x02, Connectors_Terminal_Blocks:TerminalBlock_bornier-2_P5.08mm, F.Cu at (234.4, 87.7)
- added P14: Power, Socket_Arduino_Mega:Socket_Strip_Arduino_1x08, F.Cu at (131.3, 128.3)
- added P15: Analog, Socket_Arduino_Mega:Socket_Strip_Arduino_1x08, F.Cu at (154.2, 128.5)
- added P16: Analog, Socket_Arduino_Mega:Socket_Strip_Arduino_1x08, F.Cu at (177.0, 128.5)
- added P17: Digital, Socket_Arduino_Mega:Socket_Strip_Arduino_2x18, F.Cu at (214.4, 114.0)
- added P18: PWM, Socket_Arduino_Mega:Socket_Strip_Arduino_1x10, F.Cu at (122.2, 62.2)
- added P19: PWM, Socket_Arduino_Mega:Socket_Strip_Arduino_1x08, F.Cu at (149.1, 62.2)
- added P20: Communication, Socket_Arduino_Mega:Socket_Strip_Arduino_1x08, F.Cu at (172.0, 62.2)
- added P21: CONN_01X01, Socket_Arduino_Mega:Arduino_1pin, F.Cu at (289.1, -29.5)
- added P22: CONN_01X01, Socket_Arduino_Mega:Arduino_1pin, F.Cu at (271.8, -29.5)
- added P23: CONN_01X01, Socket_Arduino_Mega:Arduino_1pin, F.Cu at (240.3, -30.2)
- added P24: CONN_01X01, Socket_Arduino_Mega:Arduino_1pin, F.Cu at (263.7, -14.2)
- added P25: CONN_01X01, Socket_Arduino_Mega:Arduino_1pin, F.Cu at (305.1, -30.0)
- added P26: CONN_01X01, Socket_Arduino_Mega:Arduino_1pin, F.Cu at (254.0, -29.5)
- added Q1: Q_PMOS_GDS, TO_SOT_Packages_SMD:TO-252-2, F.Cu at (51.7, 127.8)
- added Q2: Q_PMOS_GDS, TO_SOT_Packages_SMD:TO-252-2, F.Cu at (87.9, 52.1)
- added R1: 1K, Resistors_THT:R_Axial_DIN0207_L6.3mm_D2.5mm_P10.16mm_Horizontal, F.Cu at (73.4, 118.6)
- added R10: 50m, Resistors_THT:R_Axial_DIN0207_L6.3mm_D2.5mm_P10.16mm_Horizontal, F.Cu at (-58.3, 146.9)
- added R11: 50m, Resistors_THT:R_Axial_DIN0207_L6.3mm_D2.5mm_P10.16mm_Horizontal, F.Cu at (83.5, -0.49)
- added R12: 24K, Resistors_THT:R_Axial_DIN0207_L6.3mm_D2.5mm_P10.16mm_Horizontal, F.Cu at (-48.3, 127.3)
- added R13: 1K, Resistors_THT:R_Axial_DIN0207_L6.3mm_D2.5mm_P10.16mm_Horizontal, F.Cu at (78.3, -4.72)
- added R14: 24K, Resistors_THT:R_Axial_DIN0207_L6.3mm_D2.5mm_P10.16mm_Horizontal, F.Cu at (-21.1, 137.2)
- added R15: 1K, Resistors_THT:R_Axial_DIN0207_L6.3mm_D2.5mm_P10.16mm_Horizontal, F.Cu at (-66.9, 130.3)
- added R16: 24K, Resistors_THT:R_Axial_DIN0207_L6.3mm_D2.5mm_P10.16mm_Horizontal, F.Cu at (-92.2, 137.7)
- added R17: 1K, Resistors_THT:R_Axial_DIN0207_L6.3mm_D2.5mm_P10.16mm_Horizontal, F.Cu at (11.4, 121.4)
- added R18: 24K, Resistors_THT:R_Axial_DIN0207_L6.3mm_D2.5mm_P10.16mm_Horizontal, F.Cu at (-24.6, 86.1)
- added R19: 1K, Resistors_THT:R_Axial_DIN0207_L6.3mm_D2.5mm_P10.16mm_Horizontal, F.Cu at (-37.8, 76.2)
- added R2: 1K, Resistors_THT:R_Axial_DIN0207_L6.3mm_D2.5mm_P10.16mm_Horizontal, F.Cu at (67.1, 61.5)
- added R20: 24K, Resistors_THT:R_Axial_DIN0207_L6.3mm_D2.5mm_P10.16mm_Horizontal, F.Cu at (-51.2, 120.4)
- added R21: 1K, Resistors_THT:R_Axial_DIN0207_L6.3mm_D2.5mm_P10.16mm_Horizontal, F.Cu at (-69.8, 142.0)
- added R22: 24K, Resistors_THT:R_Axial_DIN0207_L6.3mm_D2.5mm_P10.16mm_Horizontal, F.Cu at (-61.0, 53.3)
- added R23: 1K, Resistors_THT:R_Axial_DIN0207_L6.3mm_D2.5mm_P10.16mm_Horizontal, F.Cu at (-68.3, 138.1)
- added R24: 24K, Resistors_THT:R_Axial_DIN0207_L6.3mm_D2.5mm_P10.16mm_Horizontal, F.Cu at (-25.9, -9.65)
- added R25: 1K, Resistors_THT:R_Axial_DIN0207_L6.3mm_D2.5mm_P10.16mm_Horizontal, F.Cu at (-50.5, 63.5)
- added R26: 24K, Resistors_THT:R_Axial_DIN0207_L6.3mm_D2.5mm_P10.16mm_Horizontal, F.Cu at (-71.2, 149.9)
- added R27: 1K, Resistors_THT:R_Axial_DIN0207_L6.3mm_D2.5mm_P10.16mm_Horizontal, F.Cu at (-56.9, -5.08)
- added R28: 24K, Resistors_THT:R_Axial_DIN0207_L6.3mm_D2.5mm_P10.16mm_Horizontal, F.Cu at (80.5, -16.3)
- added R29: 1K, Resistors_THT:R_Axial_DIN0207_L6.3mm_D2.5mm_P10.16mm_Horizontal, F.Cu at (-16.5, -18.0)
- added R3: 50m, Resistors_THT:R_Axial_DIN0207_L6.3mm_D2.5mm_P10.16mm_Horizontal, F.Cu at (-65.3, 34.5)
- added R30: 24K, Resistors_THT:R_Axial_DIN0207_L6.3mm_D2.5mm_P10.16mm_Horizontal, F.Cu at (4.32, -17.3)
- added R31: 1K, Resistors_THT:R_Axial_DIN0207_L6.3mm_D2.5mm_P10.16mm_Horizontal, F.Cu at (-54.6, 13.7)
- added R32: 24K, Resistors_THT:R_Axial_DIN0207_L6.3mm_D2.5mm_P10.16mm_Horizontal, F.Cu at (24.1, -17.3)
- added R33: 1K, Resistors_THT:R_Axial_DIN0207_L6.3mm_D2.5mm_P10.16mm_Horizontal, F.Cu at (56.9, -18.3)
- added R34: 1K, Resistors_THT:R_Axial_DIN0207_L6.3mm_D2.5mm_P10.16mm_Horizontal, F.Cu at (-31.8, 19.1)
- added R35: 1K, Resistors_THT:R_Axial_DIN0207_L6.3mm_D2.5mm_P10.16mm_Horizontal, F.Cu at (-12.7, 62.2)
- added R36: 1K, Resistors_THT:R_Axial_DIN0207_L6.3mm_D2.5mm_P10.16mm_Horizontal, F.Cu at (-61.2, 140.1)
- added R37: 1K, Resistors_THT:R_Axial_DIN0207_L6.3mm_D2.5mm_P10.16mm_Horizontal, F.Cu at (-34.5, 169.7)
- added R38: 1K, Resistors_THT:R_Axial_DIN0207_L6.3mm_D2.5mm_P10.16mm_Horizontal, F.Cu at (-20.3, 55.1)
- added R39: 1K, Resistors_THT:R_Axial_DIN0207_L6.3mm_D2.5mm_P10.16mm_Horizontal, F.Cu at (-27.2, 42.7)
- added R4: 50m, Resistors_THT:R_Axial_DIN0207_L6.3mm_D2.5mm_P10.16mm_Horizontal, F.Cu at (-49.3, 20.3)
- added R40: 1K, Resistors_THT:R_Axial_DIN0207_L6.3mm_D2.5mm_P10.16mm_Horizontal, F.Cu at (-36.1, 5.08)
- added R41: R, Resistors_THT:R_Axial_DIN0207_L6.3mm_D2.5mm_P10.16mm_Horizontal, F.Cu at (-76.9, 151.8)
- added R42: 220, Resistors_THT:R_Axial_DIN0207_L6.3mm_D2.5mm_P10.16mm_Horizontal, F.Cu at (104.1, -18.8)
- added R43: 1K, Resistors_THT:R_Axial_DIN0207_L6.3mm_D2.5mm_P10.16mm_Horizontal, F.Cu at (63.2, 112.8)
- added R44: 1K, Resistors_THT:R_Axial_DIN0207_L6.3mm_D2.5mm_P10.16mm_Horizontal, F.Cu at (77.2, 67.3)
- added R5: 50m, Resistors_THT:R_Axial_DIN0207_L6.3mm_D2.5mm_P10.16mm_Horizontal, F.Cu at (-30.2, 31.0)
- added R6: 50m, Resistors_THT:R_Axial_DIN0207_L6.3mm_D2.5mm_P10.16mm_Horizontal, F.Cu at (-74.1, 158.7)
- added R7: 50m, Resistors_THT:R_Axial_DIN0207_L6.3mm_D2.5mm_P10.16mm_Horizontal, F.Cu at (-49.7, 129.3)
- added R8: 50m, Resistors_THT:R_Axial_DIN0207_L6.3mm_D2.5mm_P10.16mm_Horizontal, F.Cu at (-62.6, 143.0)
- added R9: 50m, Resistors_THT:R_Axial_DIN0207_L6.3mm_D2.5mm_P10.16mm_Horizontal, F.Cu at (0.51, 73.4)
- added SW1: SW_DIP_x01, Connectors_Terminal_Blocks:TerminalBlock_bornier-2_P5.08mm, F.Cu at (72.1, 129.5)
- added SW2: SW_DIP_x01, Connectors_Terminal_Blocks:TerminalBlock_bornier-2_P5.08mm, F.Cu at (67.6, 50.5)
Other:
- board outline removed
